Commit message: update

File: integ_gazebo_model/integ_description/urdf/arm.urdf.xacro (robot description, xacro)
@@ -151,5 +151,5 @@
     <transmission name="shoulder_transmission">
       <type>transmission_interface/SimpleTransmission</type>
-      <joint name="shoulder_joint">
+      <joint name="shoulder">
         <hardwareInterface>hardware_interface/EffortJointInterface</hardwareInterface>
       </joint>
@@ -186,5 +186,5 @@
     <transmission name="elbow_transmission">
       <type>transmission_interface/SimpleTransmission</type>
-      <joint name="elbow_joint">
+      <joint name="elbow">
         <hardwareInterface>hardware_interface/EffortJointInterface</hardwareInterface>
       </joint>
