Commit message: Add files via upload

File: integ_gazebo_model/integ_description/urdf/imgproc/cible.urdf (robot description, URDF)
Before this commit: robot cible_simple, 1 links, 0 joints
Links:
- removed link my_target
- added link my_target_1, mass 1.0; collision box size=0.2 0.8 0.2; visual box size=0.2 0.8 0.2
- added link my_target_2; visual box size=0.2 0.2 0.3
Joints:
- added joint joint2: type fixed, parent my_target_1, child my_target_2
