Commit message: gazebo ok

File: integ_description/urdf/scara_sw.urdf (robot description, URDF)
Before this commit: robot scara_sw, 5 links, 4 joints
Links:
- removed link ee_frame
- link link_2: mass 3.181291 -> 7.084761
Joints:
- removed joint ee_joint
- joint world_joint: origin xyz=0. 0 3 rpy=0 0. 0 -> xyz=0. 0 1. rpy=0 0. 0

File: integ_description/urdf/scara_sw.xacro (robot description, xacro)
@@ -156,4 +156,5 @@
       <actuator name="joint_1_actuator"/>
     </transmission>
+<!--
   <link name="ee_frame"/>
   <joint name="ee_joint" type="fixed">
@@ -161,5 +162,5 @@
     <parent link="link_2" />
     <child link="ee_frame" />
-  </joint>
+  </joint>-->
   <link
     name="link_2">
@@ -190,13 +191,13 @@
     </inertial> -->
   <!--    Mass and inertia friction match   -->
-     <mass
-        value="3.181291" />
-     <inertia
-        ixx="0.013725"
-        ixy="0.00"
-        ixz="0.006881"
-        iyy="0.067471"
-        iyz="0.00"
-        izz="0.2" />
+       <mass
+        value="7.084761" />
+      <inertia
+        ixx="0.147885"
+        ixy="0.0000"
+        ixz="-0.033179"
+        iyy="0.196455"
+        iyz="0.0000"
+        izz="0.055095" />
     </inertial>
     <visual>
@@ -262,11 +263,6 @@
 -->
   </joint>
-    <transmission name="joint_2_transmission">
-      <type>transmission_interface/SimpleTransmission</type>
-      <joint name="joint_2">
-        <hardwareInterface>hardware_interface/EffortJointInterface</hardwareInterface>
-        <mechanicalReduction>15</mechanicalReduction>
-      </joint>
-      <actuator name="joint_2_actuator"/>
-    </transmission>
+    <gazebo>
+        <plugin filename="libignition-gazebo-joint-state-publisher-system.so" name="ignition::gazebo::systems::JointStatePublisher"/>
+</gazebo>
 </robot>
