Commit message: add position and velocity control for Gazebo

File: integ_description/urdf/scara_sw.xacro (robot description, xacro)
@@ -5,17 +5,33 @@
      After generation, multiple changes and additions were required as described in the 2R Robot Modeling Technical Report.-->
 <robot  name="scara_sw" xmlns:xacro="http://www.ros.org/wiki/xacro" >
- <xacro:arg name="offset" default="1."/>
+    <xacro:arg name="offset" default="1."/>
+    <xacro:arg name="mode" default="position"/>
+    <xacro:property name="mode" value="$(arg mode)"/>
     <!-- 	___________Joints Control in Gazebo___________-->
-  <gazebo>
-    <plugin name="gazebo_ros_control" filename="libgazebo_ros_control.so"/>
-  </gazebo>
-  <!-- Note that material tags supplied by SolidWorks are used in rviz but ignored by Gazebo -->
-  <gazebo reference="link_1">
-    <material>Gazebo/Turquoise</material>
-  </gazebo>
-  <gazebo reference="link_2">
-    <material>Gazebo/Orange</material>
-  </gazebo>
-  <!-- Used for fixing robot to Gazebo 'base_link' -->
+   <xacro:macro name="joint_controller" params="joint p i d cmd_max">
+    <xacro:if value="${mode == 'position'}">
+      <plugin filename="libignition-gazebo-joint-position-controller-system.so" name="ignition::gazebo::systems::JointPositionController">
+              <joint_name>${joint}</joint_name>
+              <p_gain>${p}</p_gain>
+              <i_gain>${i}</i_gain>
+              <d_gain>${d}</d_gain>
+              <i_max>${cmd_max}</i_max>
+              <i_min>${-cmd_max}</i_min>
+              <cmd_max>${cmd_max}</cmd_max>
+              <cmd_min>${-cmd_max}</cmd_min>
+          </plugin>
+    </xacro:if>
+    <xacro:if value="${mode == 'velocity'}">
+            <plugin filename="libignition-gazebo-joint-controller-system.so" name="ignition::gazebo::systems::JointController">
+              <joint_name>${joint}</joint_name>
+              <topic>${joint}_cmd_vel</topic>
+          </plugin>
+    </xacro:if>
+   </xacro:macro>
+   <gazebo>
+    <xacro:joint_controller joint="joint_1" cmd_max="30" p="700" i="0.01" d="10"/>
+    <xacro:joint_controller joint="joint_2" cmd_max="30" p="700" i="0.01" d="10"/>
+   </gazebo>
+  <!-- Used for fixing robot to Gazebo base_link -->
   <link name="world"/>
   <joint name="world_joint" type="fixed">

Commit message: add effort control

File: integ_description/urdf/scara_sw.xacro (robot description, xacro)
@@ -28,4 +28,9 @@
           </plugin>
     </xacro:if>
+    <xacro:if value="${mode == 'effort'}">
+        <plugin filename="libignition-gazebo-apply-joint-force-system.so" name="ignition::gazebo::systems::ApplyJointForce">
+          <joint_name>${joint}</joint_name>
+        </plugin>
+    </xacro:if>
    </xacro:macro>
    <gazebo>
@@ -38,7 +43,7 @@
 	<origin xyz="0. 0 $(arg offset)" rpy="0 0. 0"/>
     <parent link="world"/>
-    <child link="base_link"/>
-  </joint>
-  <link name="base_link">
+    <child link="scara/base_link"/>
+  </joint>
+  <link name="scara/base_link">
     <inertial>
        <origin
@@ -79,6 +84,5 @@
     </collision>
   </link>
-  <link
-    name="link_1">
+  <link name="scara/link_1">
     <inertial>
       <origin
@@ -135,8 +139,6 @@
       xyz="0 0 0.049"
       rpy="0 0 -1.57079632679" />
-    <parent
-      link="base_link" />
-    <child
-      link="link_1" />
+    <parent link="scara/base_link" />
+    <child link="scara/link_1" />
     <axis
       xyz="0 0 1" />
@@ -172,13 +174,11 @@
       <actuator name="joint_1_actuator"/>
     </transmission>
-<!--
-  <link name="ee_frame"/>
+  <link name="scara/ee_frame"/>
   <joint name="ee_joint" type="fixed">
   <origin xyz="0.28002 0.0 0.071" />
-    <parent link="link_2" />
-    <child link="ee_frame" />
-  </joint>-->
-  <link
-    name="link_2">
+    <parent link="scara/link_2" />
+    <child link="scara/ee_frame" />
+  </joint>
+  <link name="scara/link_2">
     <inertial>
       <origin
@@ -251,10 +251,7 @@
       xyz="0.28002 0.0 0.071"
       rpy="0 0 0" />
-    <parent
-      link="link_1" />
-    <child
-      link="link_2" />
-    <axis
-      xyz="0 0 1" />
+    <parent link="scara/link_1" />
+    <child link="scara/link_2" />
+    <axis xyz="0 0 1" />
 <!-- Velocity limit from motor max 691Rad/s  divided by Nr=15 -->
 <!-- Effort limit nominal 2Nm (Abs max=4) from motor spec times Nr=15

Commit message: Update scara_sw.xacro
On a rectifié les paramètres inertiels de link_2

File: integ_description/urdf/scara_sw.xacro (robot description, xacro)
@@ -196,5 +196,5 @@
         iyz="0.00"
         izz="0.57501" /> -->
-  <!--    Mass and inertia original
+  <!--  Mass and inertia original   -->
      <mass
         value="3.181291" />
@@ -206,7 +206,7 @@
         iyz="0.00"
         izz="0.057501" />
-    </inertial> -->
+    </inertial>
   <!--    Mass and inertia friction match   -->
-       <mass
+<!--  <mass
         value="7.084761" />
       <inertia
@@ -217,5 +217,5 @@
         iyz="0.0000"
         izz="0.055095" />
-    </inertial>
+    </inertial>  -->
     <visual>
       <origin

Commit message: Update scara_sw.xacro
Rectification des paramètres du link_1.

File: integ_description/urdf/scara_sw.xacro (robot description, xacro)
@@ -144,17 +144,16 @@
     <axis
       xyz="0 0 1" />
-<!-- Velocity limit from motor max 691Rad/s  divided by Nr=15 -->
-<!-- Effort limit nominal 2Nm (Abs max=4Nm) from motor spec times Nr=15
+<!-- Velocity limit from motor max 691Rad/s  divided by Nr=15 (= 46.07) -->
+<!-- Effort limit nominal 2Nm (Abs max=4Nm) from motor spec times Nr=15 -->
     <limit
       lower="-3.211405854"
       upper="0.0698132"
       effort="30"
-      velocity="46.1" />
--->
-    <limit
-      lower="-3.1"
-      upper="0"
-      effort="30"
-     velocity="100" />
+      velocity="46.07" />
+<!--<limit
+      lower="-3.211405854"
+      upper="0.0698132"
+      effort="100"
+      velocity="10" /> -->
  <!--    Very large friction
 	<dynamics

Commit message: Update scara_sw.xacro
On revient au code initial car les nouvelles valeurs ne sont pas bien accueillies par gazebo...

File: integ_description/urdf/scara_sw.xacro (robot description, xacro)
@@ -49,13 +49,13 @@
     <inertial>
        <origin
-         xyz="-0.00017 -0.1379088 0.000419"
+         xyz="0 0 0"
         rpy="0 0 -1.57079632679" />
       <mass
         value="15.137" />
       <inertia
-        ixx="1.156125"
+        ixx="1.1651"
         ixy="0.00079443"
         ixz="-5.3686E-06"
-        iyy="1.128704"
+        iyy="1.1282"
         iyz="-0.004763"
         izz="2.2914" />
@@ -144,16 +144,17 @@
     <axis
       xyz="0 0 1" />
-<!-- Velocity limit from motor max 691Rad/s  divided by Nr=15 (= 46.07) -->
-<!-- Effort limit nominal 2Nm (Abs max=4Nm) from motor spec times Nr=15 -->
+<!-- Velocity limit from motor max 691Rad/s  divided by Nr=15 -->
+<!-- Effort limit nominal 2Nm (Abs max=4Nm) from motor spec times Nr=15
     <limit
       lower="-3.211405854"
       upper="0.0698132"
       effort="30"
-      velocity="46.07" />
-<!--<limit
-      lower="-3.211405854"
-      upper="0.0698132"
-      effort="100"
-      velocity="10" /> -->
+      velocity="46.1" />
+-->
+    <limit
+      lower="-3.1"
+      upper="0"
+      effort="30"
+     velocity="100" />
  <!--    Very large friction
 	<dynamics
@@ -195,5 +196,5 @@
         iyz="0.00"
         izz="0.57501" /> -->
-  <!--  Mass and inertia original   -->
+  <!--    Mass and inertia original
      <mass
         value="3.181291" />
@@ -205,7 +206,7 @@
         iyz="0.00"
         izz="0.057501" />
-    </inertial>
+    </inertial> -->
   <!--    Mass and inertia friction match   -->
-<!--  <mass
+       <mass
         value="7.084761" />
       <inertia
@@ -216,5 +217,5 @@
         iyz="0.0000"
         izz="0.055095" />
-    </inertial>  -->
+    </inertial>
     <visual>
       <origin
