Commit message: camera axis + image bag

File: integ_description/urdf/camera.xacro (robot description, xacro)
@@ -4,13 +4,17 @@
         <parent link="scara/ee_frame"/>
         <child link="scara/camera"/>
-        <origin xyz="0 0 0" rpy="0 0 0"/>
+        <origin xyz="0 0 0" rpy="0 ${pi/2} 0"/>
     </joint>
     <link name="scara/camera">
-    <visual>
-        <geometry>
-            <box size="0.1 0.1 0.1"/>
-        </geometry>
-        <material name="red"/>
-    </visual>
+    <inertial>
+    <mass value="0.015"/>
+    <inertia
+    ixx="0.001"
+    ixy="0.0"
+    ixz="0.0"
+    iyy="0.001"
+    iyz="0"
+    izz="0.001"/>
+    </inertial>
     </link>
     <joint name="camera_optical" type="fixed">
@@ -19,5 +23,19 @@
         <origin xyz="0 0 0" rpy="${-pi/2} 0 ${-pi/2}" />
     </joint>
-    <link name="scara/camera_optical"></link>
+    <link name="scara/camera_optical">
+    <visual>
+        <geometry>
+            <cylinder length="0.1" radius="0.02"/>
+        </geometry>
+        <material name="blue"/>
+    </visual>
+        <visual>
+            <origin xyz="0 0 0.05"/>
+        <geometry>
+            <cylinder length="0.02" radius="0.03"/>
+        </geometry>
+        <material name="blue"/>
+    </visual>
+        </link>
 <gazebo reference="scara/camera">
   <sensor name="camera" type="camera">
@@ -30,5 +48,5 @@
     </image>
     <clip>
-        <near>0.3</near>
+        <near>0.05</near>
         <far>100</far>
     </clip>

File: integ_description/urdf/scara_sw.xacro (robot description, xacro)
@@ -177,5 +177,5 @@
   <link name="scara/ee_frame"/>
   <joint name="ee_joint" type="fixed">
-  <origin xyz="0.28002 0.0 0.071" />
+  <origin xyz="0.28002 0.0 0.03" />
     <parent link="scara/link_2" />
     <child link="scara/ee_frame" />

File: integ_description/urdf/target.xacro (robot description, xacro)
@@ -2,10 +2,10 @@
 <robot name="target" xmlns:xacro="http://www.ros.org/wiki/xacro" >-
   <xacro:arg name="vel" default="1."/>
-  <xacro:property name="offset" default=".4"/>
+  <xacro:property name="offset" default=".5"/>
   <xacro:property name="radius" default=".1"/>
-  <xacro:property name="size" default=".03"/>
+  <xacro:property name="size" default=".02"/>
   <link name="world"/>
   <joint name="world_joint" type="fixed">
-	<origin xyz="0 ${-offset} 1.1" rpy="0 0. 0"/>
+	<origin xyz="0 ${-offset} 1" rpy="0 0. 0"/>
     <parent link="world"/>
     <child link="target/base_link"/>

Commit message: cleaned repo and working visual_servoing

File: integ_description/urdf/camera.xacro (robot description, xacro)
@@ -4,17 +4,13 @@
         <parent link="scara/ee_frame"/>
         <child link="scara/camera"/>
-        <origin xyz="0 0 0" rpy="0 ${pi/2} 0"/>
+        <origin xyz="0 0 0.01" rpy="0 ${pi/2} 0"/>
     </joint>
     <link name="scara/camera">
-    <inertial>
-    <mass value="0.015"/>
-    <inertia
-    ixx="0.001"
-    ixy="0.0"
-    ixz="0.0"
-    iyy="0.001"
-    iyz="0"
-    izz="0.001"/>
-    </inertial>
+    <visual>
+        <geometry>
+            <box size="0.1 0.1 0.1"/>
+        </geometry>
+        <material name="red"/>
+    </visual>
     </link>
     <joint name="camera_optical" type="fixed">
@@ -23,24 +19,11 @@
         <origin xyz="0 0 0" rpy="${-pi/2} 0 ${-pi/2}" />
     </joint>
-    <link name="scara/camera_optical">
-    <visual>
-        <geometry>
-            <cylinder length="0.1" radius="0.02"/>
-        </geometry>
-        <material name="blue"/>
-    </visual>
-        <visual>
-            <origin xyz="0 0 0.05"/>
-        <geometry>
-            <cylinder length="0.02" radius="0.03"/>
-        </geometry>
-        <material name="blue"/>
-    </visual>
-        </link>
+    <link name="scara/camera_optical"></link>
 <gazebo reference="scara/camera">
   <sensor name="camera" type="camera">
     <camera>
     <optical_frame_id>scara/camera_optical</optical_frame_id>
-    <horizontal_fov>1.047</horizontal_fov>
+    <horizontal_fov>2.094</horizontal_fov>
+    <vertical_fov>2.094</vertical_fov>
     <image>
         <width>640</width>
@@ -48,7 +31,8 @@
     </image>
     <clip>
-        <near>0.05</near>
+        <near>0.1</near>
         <far>100</far>
     </clip>
+    <focal_length>50</focal_length>
     </camera>
     <always_on>1</always_on>

File: integ_description/urdf/scara_sw.xacro (robot description, xacro)
@@ -7,5 +7,5 @@
     <xacro:arg name="offset" default="1."/>
     <xacro:arg name="mode" default="position"/>
-    <xacro:include filename="camera.xacro" />  <!--Include the camera.xacro file ADDED BY ME-->
+    <xacro:include filename="camera.xacro" />  <!--Include the camera.xacro file -->
     <xacro:property name="mode" value="$(arg mode)"/>
     <!-- 	___________Joints Control in Gazebo___________-->
@@ -36,6 +36,6 @@
    </xacro:macro>
    <gazebo>
-    <xacro:joint_controller joint="joint_1" cmd_max="30" p="700" i="0.01" d="10"/>
-    <xacro:joint_controller joint="joint_2" cmd_max="30" p="700" i="0.01" d="10"/>
+    <xacro:joint_controller joint="joint_1" cmd_max="30" p="10" i="0" d="0"/> <!-- 700 0.01 10 -->
+    <xacro:joint_controller joint="joint_2" cmd_max="30" p="10" i="0" d="0"/> <!-- 700 0.01 10 -->
    </gazebo>
   <!-- Used for fixing robot to Gazebo base_link -->
@@ -177,5 +177,5 @@
   <link name="scara/ee_frame"/>
   <joint name="ee_joint" type="fixed">
-  <origin xyz="0.28002 0.0 0.03" />
+  <origin xyz="0.28002 0.0 0.071" />
     <parent link="scara/link_2" />
     <child link="scara/ee_frame" />

File: integ_description/urdf/target.xacro (robot description, xacro)
@@ -1,8 +1,8 @@
 <?xml version="1.0"?>
-<robot name="target" xmlns:xacro="http://www.ros.org/wiki/xacro" >-
+<robot name="target" xmlns:xacro="http://www.ros.org/wiki/xacro" >
   <xacro:arg name="vel" default="1."/>
-  <xacro:property name="offset" default=".5"/>
+  <xacro:property name="offset" default=".4"/>
   <xacro:property name="radius" default=".1"/>
-  <xacro:property name="size" default=".02"/>
+  <xacro:property name="size" default=".03"/>
   <link name="world"/>
   <joint name="world_joint" type="fixed">
@@ -22,5 +22,5 @@
         iyz="-0.004763"
         izz="2.2914" />
-    </inertial>>
+    </inertial>
   </link>
   <link name="target/ball">
@@ -58,5 +58,10 @@
         <joint_name>ball</joint_name>
         <initial_velocity>$(arg vel)</initial_velocity>
-      </plugin>
+    </plugin>
+    <plugin
+        filename="libignition-gazebo-joint-state-publisher-system.so"
+        name="ignition::gazebo::systems::JointStatePublisher">
+    <!-- Parameters would go here if there were any -->
+    </plugin>
   </gazebo>
 </robot>
